File: dorji_radio/dorji_radio.kicad_sch (KiCad schematic)
At the start: 6 parts, among them U1 DRA818V, U2 STM32C011F4Px, U3 LM380N-8

Commit message: add power input for battery
Parts:
- added AE1: Antenna, symbol Device:Antenna
- added C4, C5: .1u, symbol Device:C_Small
- added C6: 1u, symbol Device:C_Small
- added J1: Conn_01x02, Connector_JST:JST_EH_S2B-EH_1x02_P2.50mm_Horizontal, symbol Connector_Generic:Conn_01x02
- added U4: LT1762-3.3, Package_SO:MSOP-8_3x3mm_P0.65mm, symbol Regulator_Linear:LT1762-3.3
Connections:
- net +5V: no longer C1.1, C2.1, U1.8 (VBAT), U2.4 (VDD)
- net GND: now also C5.2, C6.2, J1.1 (Pin_1), U4.4 (GND)
- new net: AE1.1 (A), U1.12 (ANT)
- new net: C4.2, U4.3 (BYP)
- new net +3V3: C2.1, C4.1, C5.1, U2.4 (VDD), U4.1 (OUT), U4.2 (SENSE)
- new net +3V7: C1.1, C6.1, J1.2 (Pin_2), U1.8 (VBAT), U4.5 (~{SHDN}), U4.8 (IN)
Other:
- note added: "Also, may prefer to use a physical switch to change btwn high power and lower power for the DRA818V"
- note added: "Needs power regulator and dc-dc converter for 5V source, goal is to power using a 1-cell lipo battery"
- note added: "Power Regulation and Input"
- note added: "Questsions rn are impedence matching, antenna selection, mic input and gain"
- moved on the sheet: C1, C2, C3, U2, U3
