File: usbc_lipo_charger/usbc_lipo_charger.kicad_sch (KiCad schematic)
At the start: 18 parts, among them J1 USB_C_Receptacle_PowerOnly_6P, J2 Conn_01x02, U1 MCP73833-xxx-UN

Commit message: adding comments
Other:
- note added: "Revision Notes"
- note added: "Shrinking layout footprint, add labels to status indicator lights"
Changed lines of the file:
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@@
 	(generator_version "9.0")
 	(paper "A4")
+	(text "Shrinking layout footprint, add labels to status indicator lights"
+		(exclude_from_sim no)
+		(at 105.918 178.054 0)
+		(effects
+			(font
+				(size 1.27 1.27)
+			)
+			(justify left)
+		)
+	)
+	(text "Revision Notes"
+		(exclude_from_sim no)
+		(at 110.236 168.91 0)
+		(effects
+			(font
+				(size 1.27 1.27)
+			)
+		)
+	)
 	(text "Thermal Modeling w/ NTC Resistors:\n24k = RTS + [RTP*RCOLD/(RTP+RCOLD)]\n5k  = RTS + [RTP*RHOT/(RTP+RHOT)]"
 		(exclude_from_sim no)
@@
 	(text "Added 5.1k Pulldown at USC-C terminal, sets to 5v 3A limit"
 		(exclude_from_sim no)
-		(at 111.506 176.53 0)
+		(at 105.918 173.482 0)
 		(effects
 			(font
@@
 		)
 	)
+	(polyline
+		(pts
+			(xy 101.854 166.116) (xy 101.854 197.612)
+		)
+		(stroke
+			(width 0)
+			(type default)
+		)
+	)
 	(wire
 		(pts
@@
 		)
 		(stroke
+			(width 0)
+			(type default)
+		)
+	)
+	(polyline
+		(pts
+			(xy 177.292 166.116) (xy 101.854 166.116)
+		)
+		(stroke

Commit message: revision 1, make smaller, add pcb heatsinking, label status leds
Connections:
- net GND: now also J2.1 (Pin_1); no longer J2.2 (Pin_2)
- net VBAT: now also J2.2 (Pin_2); no longer J2.1 (Pin_1)
Changed lines of the file:
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@@
 	(label "STAT1"
 		(at 109.22 93.98 0)
+		(fields_autoplaced yes)
 		(effects
 			(font
@@
 			(justify left bottom)
 		)
+		(property "Netclass" "digital_lp"
+			(at 109.22 95.25 0)
+			(effects
+				(font
+					(size 1.27 1.27)
+					(italic yes)
+				)
+				(justify left)
+				(hide yes)
+			)
+		)
 	)
 	(symbol
@@
 	(symbol
 		(lib_id "Connector_Generic:Conn_01x02")
-		(at 204.47 88.9 0)
-		(unit 1)
-		(exclude_from_sim no)
-		(in_bom yes)
-		(on_board yes)
-		(dnp no)
-		(fields_autoplaced yes)
+		(at 204.47 91.44 0)
+		(mirror x)
+		(unit 1)
+		(exclude_from_sim no)
+		(in_bom yes)
+		(on_board yes)
+		(dnp no)
 		(property "Reference" "J2"
-			(at 207.01 88.8999 0)
+			(at 207.01 91.4401 0)
 			(effects
 				(font
@@
 		)
 		(property "Value" "Conn_01x02"
-			(at 207.01 91.4399 0)
+			(at 207.01 88.9001 0)
 			(effects
 				(font
@@
 		)
 		(property "Footprint" "Connector_Molex:Molex_SPOX_5268-02A_1x02_P2.50mm_Horizontal"
-			(at 204.47 88.9 0)
+			(at 204.47 91.44 0)
 			(effects
 				(font
@@
 		)
 		(property "Datasheet" "~"
-			(at 204.47 88.9 0)
+			(at 204.47 91.44 0)
 			(effects
 				(font
@@
 		)
 		(property "Description" "Generic connector, single row, 01x02, script generated (kicad-library-utils/schlib/autogen/connector/)"
-			(at 204.47 88.9 0)
-			(effects
-				(font
+			(at 204.47 91.44 0)
+			(effects
+				(font

Commit message: update pcb image, meet manufacture requirements
Connections:
- net VBUS: no longer names the net of C1.1, D1.2 (A), D2.2 (A), D3.2 (A), J1.A9 (VBUS), J1.B9 (VBUS), U1.1 (V_{DD}), U1.2 (V_{DD})
Changed lines of the file:
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@@
-		)
-	)
-	(label "VBUS"
-		(at 133.35 88.9 0)
-		(effects
-			(font
-				(size 1.27 1.27)
-			)
-			(justify left bottom)
 		)
 	)
